File: WordClock_eagle/wordclockv0.1.sch (EAGLE design)
At the start: 39 parts, among them IC1 TLC5925, Q1 8MHz, Q2 32.768kHz, U1 MBT3906DW1T1G, U2 MBT3906DW1T1G, U3 MBT3906DW1T1G, U4 MBT3906DW1T1G, U5 MBT3906DW1T1G

Commit message: Leds are now fed by VCC_RAW instead of 3V3
Connections:
- removed net N$5: J1.1, R3.1, U$2.VIN
- new net VCC_RAW: J1.1, R3.1, U$2.VIN, U1T1.E, U1T2.E, U2T1.E, U2T2.E, U3T1.E, U3T2.E, U4T1.E, U4T2.E, U5T1.E, U5T2.E
- net VDD: no longer U1T1.E, U1T2.E, U2T1.E, U2T2.E, U3T1.E, U3T2.E, U4T1.E, U4T2.E, U5T1.E, U5T2.E

Commit message: Updated the cam file for jlcpcb. The other files are just minor changes
idk bro seems pretty sketchy
Parts:
- JP1: device pinhead:PINHD-1X11 -> pinhead:PINHD-1X12
Connections:
- removed net N$15: IC1.!OUT5, JP1.11
- removed net N$32: IC1.!OUT7, JP1.9
- removed net N$33: IC1.!OUT6, JP1.10
- new net OUT4: IC1.!OUT4, JP1.9
- new net OUT5: IC1.!OUT5, JP1.10
- new net OUT6: IC1.!OUT6, JP1.11
- new net OUT7: IC1.!OUT7, JP1.12
Changed lines of the file:
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@@
 <part name="R5" library="rcl" library_urn="urn:adsk.eagle:library:334" deviceset="R-EU_" device="M1206" package3d_urn="urn:adsk.eagle:package:23566/1" value="13k"/>
 <part name="R6" library="rcl" library_urn="urn:adsk.eagle:library:334" deviceset="R-EU_" device="M1206" package3d_urn="urn:adsk.eagle:package:23566/1" value="59k"/>
-<part name="JP1" library="pinhead" library_urn="urn:adsk.eagle:library:325" deviceset="PINHD-1X11" device="" package3d_urn="urn:adsk.eagle:package:22410/2"/>
+<part name="JP1" library="pinhead" library_urn="urn:adsk.eagle:library:325" deviceset="PINHD-1X12" device="" package3d_urn="urn:adsk.eagle:package:22487/2"/>
 <part name="JP2" library="pinhead" library_urn="urn:adsk.eagle:library:325" deviceset="PINHD-1X10" device="" package3d_urn="urn:adsk.eagle:package:22406/2"/>
 <part name="U4" library="STM32F030RCT6TR" deviceset="MBT3906DW1T1G" device=""/>
@@
 <attribute name="VALUE" x="267.97" y="41.402" size="1.778" layer="96" rot="R180"/>
 </instance>
-<instance part="JP1" gate="A" x="256.54" y="76.2">
+<instance part="JP1" gate="G$1" x="256.54" y="76.2">
 <attribute name="NAME" x="250.19" y="92.075" size="1.778" layer="95"/>
 <attribute name="VALUE" x="250.19" y="58.42" size="1.778" layer="96"/>
@@
 <segment>
 <pinref part="IC1" gate="G$1" pin="!OUT15"/>
-<pinref part="JP1" gate="A" pin="1"/>
+<pinref part="JP1" gate="G$1" pin="1"/>
 <wire x1="254" y1="88.9" x2="228.6" y2="88.9" width="0.1524" layer="91"/>
 </segment>
@@
 <segment>
 <pinref part="IC1" gate="G$1" pin="!OUT14"/>
-<pinref part="JP1" gate="A" pin="2"/>
+<pinref part="JP1" gate="G$1" pin="2"/>
 <wire x1="254" y1="86.36" x2="228.6" y2="86.36" width="0.1524" layer="91"/>
 </segment>
@@
 <segment>
 <pinref part="IC1" gate="G$1" pin="!OUT13"/>
-<pinref part="JP1" gate="A" pin="3"/>
+<pinref part="JP1" gate="G$1" pin="3"/>
 <wire x1="254" y1="83.82" x2="228.6" y2="83.82" width="0.1524" layer="91"/>
 </segment>
@@
 <segment>
 <pinref part="IC1" gate="G$1" pin="!OUT12"/>
-<pinref part="JP1" gate="A" pin="4"/>
+<pinref part="JP1" gate="G$1" pin="4"/>
 <wire x1="254" y1="81.28" x2="228.6" y2="81.28" width="0.1524" layer="91"/>
 </segment>
@@
 <segment>
 <pinref part="IC1" gate="G$1" pin="!OUT11"/>
-<pinref part="JP1" gate="A" pin="5"/>
+<pinref part="JP1" gate="G$1" pin="5"/>
 <wire x1="254" y1="78.74" x2="228.6" y2="78.74" width="0.1524" layer="91"/>
 </segment>
@@
 <segment>
 <pinref part="IC1" gate="G$1" pin="!OUT10"/>
-<pinref part="JP1" gate="A" pin="6"/>
+<pinref part="JP1" gate="G$1" pin="6"/>
 <wire x1="254" y1="76.2" x2="228.6" y2="76.2" width="0.1524" layer="91"/>
 </segment>
@@
 <segment>
 <pinref part="IC1" gate="G$1" pin="!OUT9"/>
-<pinref part="JP1" gate="A" pin="7"/>
+<pinref part="JP1" gate="G$1" pin="7"/>
 <wire x1="254" y1="73.66" x2="228.6" y2="73.66" width="0.1524" layer="91"/>
 </segment>
@@
 <segment>
 <pinref part="IC1" gate="G$1" pin="!OUT8"/>
-<pinref part="JP1" gate="A" pin="8"/>
+<pinref part="JP1" gate="G$1" pin="8"/>
 <wire x1="254" y1="71.12" x2="228.6" y2="71.12" width="0.1524" layer="91"/>
-</segment>
-</net>
-<net name="N$32" class="0">
-<segment>
-<pinref part="IC1" gate="G$1" pin="!OUT7"/>
-<wire x1="200.66" y1="71.12" x2="198.12" y2="71.12" width="0.1524" layer="91"/>
-<wire x1="198.12" y1="71.12" x2="198.12" y2="63.5" width="0.1524" layer="91"/>
-<wire x1="198.12" y1="63.5" x2="241.3" y2="63.5" width="0.1524" layer="91"/>
-<wire x1="241.3" y1="63.5" x2="241.3" y2="68.58" width="0.1524" layer="91"/>
-<pinref part="JP1" gate="A" pin="9"/>
-<wire x1="241.3" y1="68.58" x2="254" y2="68.58" width="0.1524" layer="91"/>
-</segment>
-</net>
-<net name="N$33" class="0">
-<segment>
-<pinref part="IC1" gate="G$1" pin="!OUT6"/>
-<wire x1="200.66" y1="73.66" x2="195.58" y2="73.66" width="0.1524" layer="91"/>
-<wire x1="195.58" y1="73.66" x2="195.58" y2="60.96" width="0.1524" layer="91"/>
-<wire x1="195.58" y1="60.96" x2="243.84" y2="60.96" width="0.1524" layer="91"/>
-<wire x1="243.84" y1="60.96" x2="243.84" y2="66.04" width="0.1524" layer="91"/>
-<pinref part="JP1" gate="A" pin="10"/>
-<wire x1="243.84" y1="66.04" x2="254" y2="66.04" width="0.1524" layer="91"/>
 </segment>
 </net>
@@
 <wire x1="152.4" y1="73.66" x2="154.94" y2="73.66" width="0.1524" layer="91"/>
 <label x="154.94" y="73.66" size="1.27" layer="95" xref="yes"/>
-</segment>
-</net>
-<net name="N$15" class="0">
-<segment>
-<pinref part="IC1" gate="G$1" pin="!OUT5"/>
-<wire x1="200.66" y1="76.2" x2="193.04" y2="76.2" width="0.1524" layer="91"/>
-<wire x1="193.04" y1="76.2" x2="193.04" y2="58.42" width="0.1524" layer="91"/>
-<wire x1="193.04" y1="58.42" x2="246.38" y2="58.42" width="0.1524" layer="91"/>
-<wire x1="246.38" y1="58.42" x2="246.38" y2="63.5" width="0.1524" layer="91"/>
-<pinref part="JP1" gate="A" pin="11"/>
-<wire x1="246.38" y1="63.5" x2="254" y2="63.5" width="0.1524" layer="91"/>
 </segment>
 </net>
@@
 </segment>
 </net>
+<net name="OUT4" class="0">
+<segment>
+<pinref part="JP1" gate="G$1" pin="9"/>
+<wire x1="241.3" y1="68.58" x2="254" y2="68.58" width="0.1524" layer="91"/>
+<label x="241.3" y="68.58" size="1.27" layer="95" rot="R180" xref="yes"/>
+</segment>
+<segment>
+<pinref part="IC1" gate="G$1" pin="!OUT4"/>
+<wire x1="200.66" y1="78.74" x2="195.58" y2="78.74" width="0.1524" layer="91"/>
+<label x="195.58" y="78.74" size="1.27" layer="95" rot="R180" xref="yes"/>
+</segment>
+</net>
+<net name="OUT5" class="0">
+<segment>
+<pinref part="JP1" gate="G$1" pin="10"/>
+<wire x1="241.3" y1="66.04" x2="254" y2="66.04" width="0.1524" layer="91"/>
+<label x="241.3" y="66.04" size="1.27" layer="95" rot="R180" xref="yes"/>
+</segment>
+<segment>
+<pinref part="IC1" gate="G$1" pin="!OUT5"/>
+<wire x1="200.66" y1="76.2" x2="195.58" y2="76.2" width="0.1524" layer="91"/>
+<label x="195.58" y="76.2" size="1.27" layer="95" rot="R180" xref="yes"/>
+</segment>
+</net>
+<net name="OUT6" class="0">
+<segment>
+<pinref part="JP1" gate="G$1" pin="11"/>
+<wire x1="241.3" y1="63.5" x2="254" y2="63.5" width="0.1524" layer="91"/>
+<label x="241.3" y="63.5" size="1.27" layer="95" rot="R180" xref="yes"/>
+</segment>
+<segment>
+<pinref part="IC1" gate="G$1" pin="!OUT6"/>
+<wire x1="200.66" y1="73.66" x2="195.58" y2="73.66" width="0.1524" layer="91"/>
+<label x="195.58" y="73.66" size="1.27" layer="95" rot="R180" xref="yes"/>
+</segment>
+</net>
+<net name="OUT7" class="0">
+<segment>
+<pinref part="JP1" gate="G$1" pin="12"/>
+<wire x1="254" y1="60.96" x2="241.3" y2="60.96" width="0.1524" layer="91"/>
+<label x="241.3" y="60.96" size="1.27" layer="95" rot="R180" xref="yes"/>
+</segment>
+<segment>
+<pinref part="IC1" gate="G$1" pin="!OUT7"/>
+<wire x1="200.66" y1="71.12" x2="195.58" y2="71.12" width="0.1524" layer="91"/>
+<label x="195.58" y="71.12" size="1.27" layer="95" rot="R180" xref="yes"/>
+</segment>
+</net>

Commit message: Fixing huge error with stm32 pinout. Also revising board
My package was numbered differently than the diagram in the datasheet. Didn't realize until the thing was hot to the touch and not responding. sucks to be me
Parts:
- U$1: value STM32F030RCT6TR -> STM32F030RCT6TRLQFP64; device STM32F030RCT6TR:STM32F030RCT6TR -> STM32F030RCT6TR:STM32F030RCT6TRLQFP64
Changed lines of the file:
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@@
 <part name="Q2" library="crystal" deviceset="CRYSTAL" device="TC26V" value="32.768kHz"/>
 <part name="Q1" library="crystal" library_urn="urn:adsk.eagle:library:204" deviceset="CRYSTAL" device="HC49U-V" package3d_urn="urn:adsk.eagle:package:12075/1" value="8MHz"/>
-<part name="U$1" library="STM32F030RCT6TR" deviceset="STM32F030RCT6TR" device=""/>
+<part name="U$1" library="STM32F030RCT6TR" deviceset="STM32F030RCT6TR" device="LQFP64"/>
 <part name="U$2" library="STM32F030RCT6TR" deviceset="AP65111A" device=""/>
 <part name="R3" library="rcl" library_urn="urn:adsk.eagle:library:334" deviceset="R-EU_" device="M1206" package3d_urn="urn:adsk.eagle:package:23566/1" value="100k"/>
